Commit message: Added a diff_params.yaml file for params.

File: nuturtle_description/urdf/turtlebot3_burger.urdf.xacro (robot description, xacro)
@@ -3,4 +3,9 @@
   xmlns:xacro="http://ros.org/wiki/xacro">
   <!-- <xacro:include filename="$(find turtlebot3_description)/urdf/common_properties.urdf"/> -->
+  <xacro:property name="ddrive_params" value="$(find nuturtle_description)/config/diff_params.yaml" />
+  <xacro:property name="params" value="${xacro.load_yaml(ddrive_params)['ros__parameters']}" />
+  <xacro:property name="wheel_radius"  value="${params['wheel_radius']}" />
+  <xacro:property name="track_width"  value="${params['track_width']}" />
+  <xacro:property name="collision_radius"  value="${params['collision_radius']}" />
   <!-- Init colour -->
   <material name="black">
@@ -63,5 +68,5 @@
     <parent link="base_link"/>
     <child link="wheel_left_link"/>
-    <origin xyz="0.0 0.08 0.023" rpy="-1.57 0 0"/>
+    <origin xyz="0.0 ${(track_width)/2} 0.023" rpy="-1.57 0 0"/>
     <axis xyz="0 0 1"/>
   </joint>
@@ -77,5 +82,5 @@
       <origin xyz="0 0 0" rpy="0 0 0"/>
       <geometry>
-        <cylinder length="0.018" radius="0.033"/>
+        <cylinder length="0.018" radius="${wheel_radius}"/>
       </geometry>
     </collision>
@@ -89,5 +94,5 @@
     <parent link="base_link"/>
     <child link="wheel_right_link"/>
-    <origin xyz="0.0 -0.080 0.023" rpy="-1.57 0 0"/>
+    <origin xyz="0.0 -${(track_width)/2} 0.023" rpy="-1.57 0 0"/>
     <axis xyz="0 0 1"/>
   </joint>
@@ -103,5 +108,5 @@
       <origin xyz="0 0 0" rpy="0 0 0"/>
       <geometry>
-        <cylinder length="0.018" radius="0.033"/>
+        <cylinder length="0.018" radius="${wheel_radius}"/>
       </geometry>
     </collision>

Commit message: Modified collision radius for the base link.
Full functionality as expected in Task A.3

File: nuturtle_description/urdf/turtlebot3_burger.urdf.xacro (robot description, xacro)
@@ -53,10 +53,20 @@
       <material name="light_black"/>
     </visual>
-    <collision>
-      <origin xyz="-0.032 0 0.070" rpy="0 0 0"/>
-      <geometry>
-        <box size="0.140 0.140 0.143"/>
-      </geometry>
-    </collision>
+    <xacro:if value="${collision_radius &gt; 0}">
+      <collision>
+        <origin xyz="-0.032 0 0.070" rpy="0 0 0"/>
+        <geometry>
+          <cylinder length="0.143" radius="${collision_radius}"/>
+        </geometry>
+      </collision>
+    </xacro:if>
+    <xacro:if value="${collision_radius &lt; 0}">
+      <collision>
+        <origin xyz="-0.032 0 0.070" rpy="0 0 0"/>
+        <geometry>
+          <box size="0.140 0.140 0.143"/>
+        </geometry>
+      </collision>
+    </xacro:if>
     <inertial>
       <origin xyz="0 0 0" rpy="0 0 0"/>

Commit message: Full functionality as expected in Task A4.
Added color argument to the xacro file. Added
rviz config files for each color.

File: nuturtle_description/urdf/turtlebot3_burger.urdf.xacro (robot description, xacro)
@@ -8,5 +8,9 @@
   <xacro:property name="track_width"  value="${params['track_width']}" />
   <xacro:property name="collision_radius"  value="${params['collision_radius']}" />
+  <xacro:arg name="color" default="purple"/>
   <!-- Init colour -->
+  <material name="purple">
+      <color rgba="0.3 0.16 0.52 1.0"/>
+  </material>
   <material name="black">
       <color rgba="0.0 0.0 0.0 1.0"/>
@@ -51,5 +55,5 @@
         <mesh filename="package://nuturtle_description/meshes/burger_base.stl" scale="0.001 0.001 0.001"/>
       </geometry>
-      <material name="light_black"/>
+      <material name="$(arg color)"/>
     </visual>
     <xacro:if value="${collision_radius &gt; 0}">

Commit message: Implemented sim control using teleop

File: nuturtle_description/urdf/turtlebot3_burger.urdf.xacro (robot description, xacro)
@@ -4,5 +4,5 @@
   <!-- <xacro:include filename="$(find turtlebot3_description)/urdf/common_properties.urdf"/> -->
   <xacro:property name="ddrive_params" value="$(find nuturtle_description)/config/diff_params.yaml" />
-  <xacro:property name="params" value="${xacro.load_yaml(ddrive_params)['ros__parameters']}" />
+  <xacro:property name="params" value="${xacro.load_yaml(ddrive_params)['/**']['ros__parameters']}" />
   <xacro:property name="wheel_radius"  value="${params['wheel_radius']}" />
   <xacro:property name="track_width"  value="${params['track_width']}" />
